File: tara-keyboard/tara-keyboard.kicad_pcb (KiCad board)
At the start: 4 copper layers, 349 x 126 mm, 202 parts, among them J1 USB_C_Receptacle_USB2.0_14P, J2 BOOT, SW1 RST, U1 STM32F072RBTx, U2 USBLC6-2SC6, U3 XC6220B331MR

Commit message: :construction: work in progress.
Parts:
- removed the REF** at (285.0, 115.7)
- removed the REF** at (46.9, 115.7)
- added D89: CAPS, LED_SMD:LED_0603_1608Metric, F.Cu at (389.1, 112.2)
- added J3: Conn_01x05, Connector_PinHeader_2.54mm:PinHeader_1x05_P2.54mm_Vertical, F.Cu at (381.3, 129.4)
- added R7: 510R, Resistor_SMD:R_0402_1005Metric, F.Cu at (389.1, 113.5)
- added REF**: Stabilizer_Cherry_MX_2.00u, PCM_Mounting_Keyboard_Stabilizer:Stabilizer_Cherry_MX_2.00u, F.Cu at (288.1, 123.8)
- added REF**: Stabilizer_Cherry_MX_2.00u, PCM_Mounting_Keyboard_Stabilizer:Stabilizer_Cherry_MX_2.00u, F.Cu at (50.0, 123.8)
- added REF**: Stabilizer_Cherry_MX_2.00u, PCM_Mounting_Keyboard_Stabilizer:Stabilizer_Cherry_MX_2.00u, F.Cu at (295.3, 66.7)
- added REF**: Stabilizer_Cherry_MX_2.00u, PCM_Mounting_Keyboard_Stabilizer:Stabilizer_Cherry_MX_2.00u, F.Cu at (45.2, 104.8)
- added REF**: Stabilizer_Cherry_MX_2.00u, PCM_Mounting_Keyboard_Stabilizer:Stabilizer_Cherry_MX_2.00u, F.Cu at (292.9, 104.8)
- C1: value 100n -> 10u; footprint Capacitor_SMD:C_0402_1005Metric -> Capacitor_SMD:C_1206_3216Metric
- C8: value 10u -> 100n; footprint Capacitor_SMD:C_1206_3216Metric -> Capacitor_SMD:C_0402_1005Metric
- J2: footprint Connector_PinHeader_2.54mm:PinHeader_1x02_P2.54mm_Horizontal -> Connector_PinHeader_2.54mm:PinHeader_1x02_P2.54mm_Vertical
- R1, R2: value 10K -> 5K1
- R3, R4: value 5K1 -> 10K
- U1: value STM32F072RBTx -> USBLC6-2SC6; footprint Package_QFP:LQFP-64_10x10mm_P0.5mm -> Package_TO_SOT_SMD:SOT-23-6
- U2: value USBLC6-2SC6 -> STM32F072RBTx; footprint Package_TO_SOT_SMD:SOT-23-6 -> Package_QFP:LQFP-64_10x10mm_P0.5mm
- moved C2 55.9 mm to (370.6, 112.0), turned to -90 degrees
- moved C7 52.5 mm to (320.0, 127.0), turned to 90 degrees
- moved C1 49.1 mm to (362.6, 102.0), turned to 90 degrees
- moved U2 46.5 mm to (327.3, 123.0), turned to 90 degrees
- moved U1 44.5 mm to (365.8, 102.0), turned to 90 degrees
- moved C8 41.3 mm to (334.6, 126.3), turned to -90 degrees
- moved R6 33.6 mm to (382.1, 113.8), turned to 0 degrees
- moved R4 33.0 mm to (370.2, 120.8), turned to 90 degrees
- moved D88 31.6 mm to (382.1, 112.5), turned to 180 degrees
- moved C5 23.5 mm to (324.1, 130.3), turned to 0 degrees
- moved R2 19.4 mm to (369.0, 96.2), turned to 180 degrees
- moved C6 15.6 mm to (329.3, 130.3), turned to 180 degrees
- moved R3 12.5 mm to (369.5, 112.0), turned to -90 degrees
- moved D35 8.95 mm to (69.8, 89.5)
- moved D36 8.95 mm to (88.9, 89.5)
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Connections:
- C1 pad 1: +3V3 -> +5V
- C2 pad 1: +3V3 -> NRST
- C7 pad 1: NRST -> +3V3
- C8 pad 1: +5V -> +3V3
- D1 pad 1: COL1 -> ROW1
- D10 pad 1: COL1 -> ROW1
- D11 pad 1: COL1 -> ROW1
- D12 pad 1: COL1 -> ROW1
- D13 pad 1: COL1 -> ROW1
- D14 pad 1: COL1 -> ROW1
- D15 pad 1: COL1 -> ROW1
- D16 pad 1: COL1 -> ROW1
- D2 pad 1: COL1 -> ROW1
- D3 pad 1: COL1 -> ROW1
- D4 pad 1: COL1 -> ROW1
- D5 pad 1: COL1 -> ROW1
- D6 pad 1: COL1 -> ROW1
- D7 pad 1: COL1 -> ROW1
- D8 pad 1: COL1 -> ROW1
- D9 pad 1: COL1 -> ROW1
- MX10 pad 1: COL10 -> COL11
- MX11 pad 1: COL11 -> COL12
- MX12 pad 1: COL12 -> COL13
- MX13 pad 1: COL13 -> COL14
- MX14 pad 1: COL14 -> COL15
- MX15 pad 1: COL15 -> COL16
- MX16 pad 1: COL16 -> COL17
- MX17 pad 1: unconnected-(MX17-Pad1) -> COL1
- MX18 pad 1: COL1 -> COL2
- MX19 pad 1: COL2 -> COL3
- MX2 pad 1: COL2 -> COL3
- MX20 pad 1: COL3 -> COL4
- MX21 pad 1: COL4 -> COL5
- MX22 pad 1: COL5 -> COL6
- MX23 pad 1: COL6 -> COL7
- MX24 pad 1: COL7 -> COL8
- MX25 pad 1: COL8 -> COL9
- MX26 pad 1: COL9 -> COL10
- MX27 pad 1: COL10 -> COL11
- MX28 pad 1: COL11 -> COL12
- MX29 pad 1: COL12 -> COL13
- MX3 pad 1: COL3 -> COL4
- MX30 pad 1: COL13 -> COL14
- MX31 pad 1: COL14 -> COL15
- MX32 pad 1: COL15 -> COL16
- MX33 pad 1: COL16 -> COL17
- MX34 pad 1: unconnected-(MX34-Pad1) -> COL1
- MX35 pad 1: COL1 -> COL2
- MX36 pad 1: COL2 -> COL3
- MX37 pad 1: COL3 -> COL4
- MX38 pad 1: COL4 -> COL5
- MX39 pad 1: COL5 -> COL6
- MX4 pad 1: COL4 -> COL5
- MX40 pad 1: COL6 -> COL7
- MX41 pad 1: COL7 -> COL8
- MX42 pad 1: COL8 -> COL9
- MX43 pad 1: COL9 -> COL10
- MX44 pad 1: COL10 -> COL11
- MX45 pad 1: COL11 -> COL12
- MX46 pad 1: COL12 -> COL13
- MX47 pad 1: COL13 -> COL14
- MX48 pad 1: COL14 -> COL15
- MX49 pad 1: COL15 -> COL16
- MX5 pad 1: COL5 -> COL6
- MX50 pad 1: COL16 -> COL17
- MX51 pad 1: COL4 -> COL1
- MX52 pad 1: COL5 -> COL2
- MX53 pad 1: COL6 -> COL3
- MX54 pad 1: COL7 -> COL4
- MX55 pad 1: COL8 -> COL5
- MX56 pad 1: COL9 -> COL6
- MX57 pad 1: COL10 -> COL7
- MX58 pad 1: COL11 -> COL8
- MX59 pad 1: COL12 -> COL9
- MX6 pad 1: COL6 -> COL7
- MX60 pad 1: COL13 -> COL10
- MX61 pad 1: COL14 -> COL11
- MX62 pad 1: COL15 -> COL12
- MX63 pad 1: COL16 -> COL14
- MX64 pad 1: COL4 -> COL1
- MX65 pad 1: COL5 -> COL2
- MX66 pad 1: COL6 -> COL3
- MX67 pad 1: COL7 -> COL4
- MX68 pad 1: COL8 -> COL5
- MX69 pad 1: COL9 -> COL6
- MX7 pad 1: COL7 -> COL8
- MX70 pad 1: COL10 -> COL7
- MX71 pad 1: COL11 -> COL8
- MX72 pad 1: COL12 -> COL9
- MX73 pad 1: COL13 -> COL10
- MX74 pad 1: COL14 -> COL11
- MX75 pad 1: COL15 -> COL14
- MX77 pad 1: COL6 -> COL1
- MX78 pad 1: COL7 -> COL2
- MX79 pad 1: COL8 -> COL3
- MX8 pad 1: COL8 -> COL9
- MX80 pad 1: COL9 -> COL6
- MX83 pad 1: COL12 -> COL13
- MX84 pad 1: COL13 -> COL14
- MX85 pad 1: COL14 -> COL15
- MX86 pad 1: COL15 -> COL16
- MX87 pad 1: COL16 -> COL17
- MX9 pad 1: COL9 -> COL10
- R1 pad 1: NRST -> Net-(J1-CC1)
- R1 pad 2: +3V3 -> GND
- R2 pad 1: GND -> Net-(J1-CC2)
- R2 pad 2: BOOT0 -> GND
- R3 pad 1: Net-(J1-CC1) -> NRST
- R3 pad 2: GND -> +3V3
- R4 pad 1: Net-(J1-CC2) -> GND
- R4 pad 2: GND -> BOOT0
- U1 pad 1: +3V3 -> USB_N
- U1 pad 2: unconnected-(U1-PC13-Pad2) -> GND
- U1 pad 3: unconnected-(U1-PC14-Pad3) -> USB_P
- U1 pad 4: unconnected-(U1-PC15-Pad4) -> USB_P
- U1 pad 5: unconnected-(U1-PF0-Pad5) -> +5V
- U1 pad 6: unconnected-(U1-PF1-Pad6) -> USB_N
- U2 pad 1: USB_N -> +3V3
- U2 pad 2: GND -> unconnected-(U2-PC13-Pad2)
- U2 pad 3: USB_P -> unconnected-(U2-PC14-Pad3)
- U2 pad 4: USB_P -> unconnected-(U2-PC15-Pad4)
- U2 pad 5: +5V -> unconnected-(U2-PF0-Pad5)
- U2 pad 6: USB_N -> unconnected-(U2-PF1-Pad6)
Routing:
- net COL1: track 0.00 -> 427.9 mm
- net ROW1: track 0.00 -> 412.9 mm, vias 0 -> 1
- net ROW2: track 0.00 -> 386.7 mm, vias 0 -> 1
- net COL2: track 0.00 -> 386.3 mm
- net COL3: track 0.00 -> 384.6 mm
- net ROW3: track 0.00 -> 362.0 mm, vias 0 -> 1
- net ROW6: track 0.00 -> 360.4 mm, vias 0 -> 1
- net COL4: track 0.00 -> 348.3 mm
- net ROW5: track 0.00 -> 331.3 mm, vias 0 -> 1
- net COL5: track 0.00 -> 329.4 mm
- net COL6: track 0.00 -> 306.2 mm
- net ROW4: track 0.00 -> 282.7 mm, vias 0 -> 1
- net COL11: track 0.00 -> 220.9 mm, vias 0 -> 1
- net COL14: track 0.00 -> 192.7 mm, vias 0 -> 1
- net COL13: track 0.00 -> 183.3 mm, vias 0 -> 2
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Other:
- board size 349 x 126 mm -> 347.8 x 123.9 mm
