File: tara-keyboard/tara-keyboard.kicad_sch (KiCad schematic)
At the start: 199 parts, among them J1 USB_C_Receptacle_USB2.0_14P, J2 BOOT, SW1 RST, U1 STM32F072RBTx, U2 USBLC6-2SC6, U3 XC6220B331MR

Commit message: :construction: work in progress.
Parts:
- added D89: CAPS, LED_SMD:LED_0603_1608Metric, symbol Device:LED_Small
- added J3: Conn_01x05, Connector_PinHeader_2.54mm:PinHeader_1x05_P2.54mm_Vertical, symbol Connector_Generic:Conn_01x05
- added R7: 510R, Resistor_SMD:R_0402_1005Metric, symbol Device:R_Small
- J2: footprint Connector_PinHeader_2.54mm:PinHeader_1x02_P2.54mm_Horizontal -> Connector_PinHeader_2.54mm:PinHeader_1x02_P2.54mm_Vertical
- renumbered C8 to C1, C7 to C2, C1 to C3, C2 to C4, C3 to C5, C4 to C6, C5 to C7, C6 to C8, R3 to R1, R4 to R2, R1 to R3, R2 to R4, U2 to U1, U1 to U2
Connections:
- net +5V: now also D89.2 (A), J3.1 (Pin_1)
- net COL1: now also MX17.1, MX34.1, MX51.1, MX64.1, MX77.1, U2.62 (PB9); no longer D1.1 (K), D10.1 (K), D11.1 (K), D12.1 (K), D13.1 (K), D14.1 (K), D15.1 (K), D16.1 (K), D2.1 (K), D3.1 (K), D4.1 (K), D5.1 (K), D6.1 (K), D7.1 (K), D8.1 (K), D9.1 (K), MX18.1, MX35.1
- net COL10: now also MX26.1, MX43.1, MX60.1, MX73.1, MX9.1, U2.40 (PC9); no longer MX10.1, MX27.1, MX44.1, MX57.1, MX70.1
- net COL11: now also MX10.1, MX27.1, MX44.1, MX61.1, MX74.1, U2.39 (PC8); no longer MX11.1, MX28.1, MX45.1, MX58.1, MX71.1
- net COL12: now also MX11.1, MX28.1, MX45.1, MX62.1, U2.38 (PC7); no longer MX12.1, MX29.1, MX46.1, MX59.1, MX72.1, MX83.1
- net COL13: now also MX12.1, MX29.1, MX46.1, MX83.1, U2.37 (PC6); no longer MX13.1, MX30.1, MX47.1, MX60.1, MX73.1, MX84.1
- net COL14: now also MX13.1, MX30.1, MX47.1, MX63.1, MX75.1, MX84.1, U2.36 (PB15); no longer MX14.1, MX31.1, MX48.1, MX61.1, MX74.1, MX85.1
- net COL15: now also MX14.1, MX31.1, MX48.1, MX85.1, U2.35 (PB14); no longer MX15.1, MX32.1, MX49.1, MX62.1, MX75.1, MX86.1
- net COL16: now also MX15.1, MX32.1, MX49.1, MX86.1, U2.34 (PB13); no longer MX16.1, MX33.1, MX50.1, MX63.1, MX87.1
- net COL2: now also MX18.1, MX35.1, MX52.1, MX65.1, MX78.1, U2.61 (PB8); no longer MX19.1, MX2.1, MX36.1
- net COL3: now also MX19.1, MX2.1, MX36.1, MX53.1, MX66.1, MX79.1, U2.59 (PB7); no longer MX20.1, MX3.1, MX37.1
- net COL4: now also MX20.1, MX3.1, MX37.1, MX54.1, MX67.1, U2.58 (PB6); no longer MX21.1, MX38.1, MX4.1, MX51.1, MX64.1
- net COL5: now also MX21.1, MX38.1, MX4.1, MX55.1, MX68.1, U2.57 (PB5); no longer MX22.1, MX39.1, MX5.1, MX52.1, MX65.1
- net COL6: now also MX22.1, MX39.1, MX5.1, MX56.1, MX69.1, MX80.1, U2.56 (PB4); no longer MX23.1, MX40.1, MX53.1, MX6.1, MX66.1, MX77.1
- net COL7: now also MX23.1, MX40.1, MX57.1, MX6.1, MX70.1, U2.43 (PA10); no longer MX24.1, MX41.1, MX54.1, MX67.1, MX7.1, MX78.1
- net COL8: now also MX24.1, MX41.1, MX58.1, MX7.1, MX71.1, U2.42 (PA9); no longer MX25.1, MX42.1, MX55.1, MX68.1, MX79.1, MX8.1
- net COL9: now also MX25.1, MX42.1, MX59.1, MX72.1, MX8.1, U2.41 (PA8); no longer MX26.1, MX43.1, MX56.1, MX69.1, MX80.1, MX9.1
- net GND: now also J3.5 (Pin_5), R7.1
- net NRST: now also J3.4 (Pin_4)
- net ROW2: now also U2.51 (PC10)
- net ROW3: now also U2.52 (PC11)
- net ROW4: now also U2.53 (PC12)
- net ROW5: now also U2.54 (PD2)
- net ROW6: now also U2.55 (PB3)
- net SWCLK: now also J3.2 (Pin_2)
- net SWDIO: now also J3.3 (Pin_3)
- net COL17: now reaches U2.33 (PB12)
- net COL17: now also MX16.1, MX33.1, MX50.1, MX87.1
- net ROW1: now reaches U2.50 (PA15)
- net ROW1: now also D1.1 (K), D10.1 (K), D11.1 (K), D12.1 (K), D13.1 (K), D14.1 (K), D15.1 (K), D16.1 (K), D2.1 (K), D3.1 (K), D4.1 (K), D5.1 (K), D6.1 (K), D7.1 (K), D8.1 (K), D9.1 (K)
- new net: D89.1 (K), R7.2
- no-connect marks 0 -> 24
Other:
- moved on the sheet: C10, C11, C12, C3, C4, C5, C6, C7, C8, C9, D17, D18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

Commit message: :rocket: Added finished PCB and generated Step Model.
Parts:
- added H1, H2, H3, H4, H5, H6, H7, H8: MountingHole, MountingHole:MountingHole_3.2mm_M3, symbol Mechanical:MountingHole
Connections:
- net +5V: no longer D89.2 (A)
- net SWCLK: now also J3.3 (Pin_3); no longer J3.2 (Pin_2)
- net SWDIO: now also J3.2 (Pin_2); no longer J3.3 (Pin_3)
- net CAPS: now reaches U2.29 (PB10)
- net CAPS: now also D89.2 (A)
- no-connect marks 24 -> 23
Other:
- moved on the sheet: J3, U2
